Commit message: clustering msgs and plugin viz

File: carina_description/urdf/carina2.urdf (robot description, URDF)
Before this commit: robot multipleshapes, 12 links, 11 joints
Links:
- removed link /base_laser_link
- removed link /radaresr1
- removed link /radaresr2
- removed link /radarside1
- removed link /radarside2
- removed link bumblebee
- removed link imu_link
- removed link ladybug_link
- added link stereo, mass 2; visual box size=0.0474 0.157 0.036
Joints:
- removed joint base_link_bumblebee_joint
- removed joint base_link_imu_joint
- removed joint base_link_ladybug_joint
- removed joint base_link_radar1_joint
- removed joint base_link_radar2_joint
- removed joint base_link_radarside1_joint
- removed joint base_link_radarside2_joint
- removed joint base_link_sick_joint
- added joint base_link_stereo_joint: type fixed, parent base_link, child stereo, origin xyz=0 0 2.1 rpy=-1.570796327 0 -1.570796327
- joint base_link_gps_joint: origin xyz=-0.59 0 1.27 rpy=0 0 0 -> xyz=0 0 2.1 rpy=0 0 0
- joint base_link_velodyne_joint: origin xyz=-0.30 0 1.677 rpy=0 0 0 -> xyz=0 0 2.1 rpy=0 0 0
